File: Schematic/T06_preliminarySchematic_v3.sch (EAGLE design)
At the start: 53 parts, among them Q3 2n3904, U1 ATMEGA328P_PDIP, X1 SSW-105-02-S-S

Commit message: Changed the LED package numbers. Added a Orange LED to the Reset Switch. This goes low when the reset is pressed. Fixed the bypass capacitor problems. Added 100nF bypass capacitor to the VCC and AVCC
Parts:
- added C6: 100n, eagle-ltspice:CC1005
- added LED3: LTST-C170KFKT, adafruit:LEDCHIP-LED0805
- added R7: 220, eagle-ltspice:RR0603
- added X2: SSW-102-02-S-S, con-samtec:SSW-102-02-S-S
- C3: device eagle-ltspice:CC1206 -> eagle-ltspice:CC1005
- LED1: value C566C-GFS-CV0Z0792 -> LTST-C171GKT
- LED2: value C566C-GFS-CV0Z0792 -> LTST-C171GKT; device adafruit:LEDCHIPLED_0805 -> adafruit:LEDCHIP-LED0805
- Q3: device SparkFun-DiscreteSemi:TRANSISTOR_NPNTO-92-AMMO -> SparkFun-DiscreteSemi:TRANSISTOR_NPN2N3904
Connections:
- new net N$9: LED3.A, R7.2
- net +5V: now also C6.1, X2-2.1; no longer C3.2
- net GND: now also C3.2, C6.2, LED3.C, X2-1.1
- net RESET: now also R7.1
Other:
- moved on the sheet: LED2, R3
