File: Board/T06_preliminarySchematic_v3.sch (EAGLE design)
At the start: 58 parts, among them Q3 2n3904, U1 ATMEGA328P_PDIP, X1 SSW-105-02-S-S, X2 SSW-102-02-S-S

Commit message: Changes reflected in the board. Changes made in the master branch. - Dusan
Parts:
- removed CSTCE16M0V53-R0: 16M, adafruit:CERMOSCILL-THM
- removed TP15: TPPAD1-13, testpad:TPPAD1-13
- added CSC: 16M, adafruit:CERMOSCILL-CSTCRG
- renumbered MOTOR1 to M1, MOTOR2 to M2, SONAR1 to S1, SONAR2 to S2, SONAR3 to S3
Connections:
- net ECHO3: no longer TP15.TP
- net GND: now also CSC.GND; no longer CSTCE16M0V53-R0.GND
- net N$1: now also CSC.OUT; no longer CSTCE16M0V53-R0.OUT
- net N$2: now also CSC.IN; no longer CSTCE16M0V53-R0.IN
